Commit message: started working on screw_perception.cpp

File: irb120_gripper_pkg/urdf/irb120_with_robotiq.xacro (robot description, xacro)
@@ -16,5 +16,5 @@
 	<xacro:include filename="$(find robotiq_85_description)/urdf/robotiq_85_gripper.urdf.xacro" />
 	<xacro:robotiq_85_gripper prefix="simple_gripper_" parent="simple_arm_tool0">
-		<origin xyz="0 0 0" rpy="${pi/2} -${pi/2} 0" />
+		<origin xyz="0 0 0" rpy="0 -${pi/2} 0" />
 	</xacro:robotiq_85_gripper>
 </robot>
