Commit message: update 22/12/23

File: irb120_gripper_pkg/urdf/irb120_with_robotiq_STAR.xacro (robot description, xacro)
@@ -1,16 +1,13 @@
 <?xml version="1.0"?>
-<robot xmlns:xacro="http://ros.org/wiki/xacro"
-       name="irb120_with_gripper" >
+<robot xmlns:xacro="http://ros.org/wiki/xacro" name="irb120_with_gripper" >
 	<xacro:arg name="limited" default="true"/>
-	<!-- THE ROBOT -->
-	<link name="world" />
-	<!-- irb120 from ROS-i repos -->
-	<xacro:include filename="$(find abb_irb120_support)/urdf/irb120_3_58_macro.xacro" />
-	<joint name="world_joint" type="fixed">
-		<parent link="world" />
-		<child link = "base_link" />
-		<origin xyz="0.0 0.0 0.0" rpy="0.0 0.0 0.0" />
-	</joint>
-	<xacro:abb_irb120_3_58 prefix="" />
+  	<xacro:include filename="$(find abb_irb120_gazebo)/urdf/irb120_3_58_macro.xacro"/>
+  	<xacro:abb_irb120_3_58_g prefix=""/>
+  	<!-- Fix robot to Gazebo world -->
+  	<link name="world"/>
+  	<joint name="world-base_link-fixed" type="fixed">
+    	<parent link="world"/>
+    	<child link="base_link"/>
+  	</joint>
 	<!-- Robotiq gripper-->
 	<xacro:include filename="$(find robotiq_85_description)/urdf/robotiq_85_gripper.urdf.xacro" />

File: irb120_robotiq_gazebo/urdf/irb120_robotiq_gazebo.urdf (robot description, URDF)
Before this commit: robot irb120_with_gripper, 20 links, 19 joints
Links:
- removed link simple_arm_base
- removed link simple_arm_base_link
- removed link simple_arm_flange
- removed link simple_arm_link_1
- removed link simple_arm_link_2
- removed link simple_arm_link_3
- removed link simple_arm_link_4
- removed link simple_arm_link_5
- removed link simple_arm_link_6
- removed link simple_arm_tool0
- removed link simple_gripper_robotiq_85_base_link
- removed link simple_gripper_robotiq_85_left_finger_link
- removed link simple_gripper_robotiq_85_left_finger_tip_link
- removed link simple_gripper_robotiq_85_left_inner_knuckle_link
- removed link simple_gripper_robotiq_85_left_knuckle_link
- removed link simple_gripper_robotiq_85_right_finger_link
- removed link simple_gripper_robotiq_85_right_finger_tip_link
- removed link simple_gripper_robotiq_85_right_inner_knuckle_link
- removed link simple_gripper_robotiq_85_right_knuckle_link
- added link base
- added link base_link, mass 6.215; collision mesh filename=package://abb_irb120_support/meshes/irb120_3_58/collision/b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; visual mesh filename=package://abb_irb120_support/meshes/irb120_3_58/visual/base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
- added link flange
- added link link_1, mass 3.067; collision mesh filename=package://abb_irb120_support/meshes/irb120_3_58/collision/l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; visual mesh filename=package://abb_irb120_support/meshes/irb120_3_58/visual/link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
- added link link_2, mass 3.909; collision mesh filename=package://abb_irb120_support/meshes/irb120_3_58/collision/l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; visual mesh filename=package://abb_irb120_support/meshes/irb120_3_58/visual/link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
- added link link_3, mass 2.944; collision mesh filename=package://abb_irb120_support/meshes/irb120_3_58/collision/l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; visual mesh filename=package://abb_irb120_support/meshes/irb120_3_58/visual/link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
- added link link_4, mass 1.328; collision mesh filename=package://abb_irb120_support/meshes/irb120_3_58/collision/l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; visual mesh filename=package://abb_irb120_support/meshes/irb120_3_58/visual/link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
- added link link_5, mass 0.546; collision mesh filename=package://abb_irb120_support/meshes/irb120_3_58/collision/l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; visual mesh filename=package://abb_irb120_support/meshes/irb120_3_58/visual/link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
- added link link_6, mass 0.137; collision mesh filename=package://abb_irb120_support/meshes/irb120_3_58/collision/l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; visual mesh filename=package://abb_irb120_support/meshes/irb120_3_58/visual/link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
- added link robotiq_85_base_link, mass 0.636951; collision mesh filename=package://robotiq_85_description/meshes/collision/robotiq_8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; visual mesh filename=package://robotiq_85_description/meshes/visual/robotiq_85_b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
- added link robotiq_85_left_finger_link, mass 0.027309; collision mesh filename=package://robotiq_85_description/meshes/collision/robotiq_8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; visual mesh filename=package://robotiq_85_description/meshes/visual/robotiq_85_f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
- added link robotiq_85_left_finger_tip_link, mass 0.019555; collision mesh filename=package://robotiq_85_description/meshes/collision/robotiq_8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; visual mesh filename=package://robotiq_85_description/meshes/visual/robotiq_85_f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
- added link robotiq_85_left_inner_knuckle_link, mass 0.029951; collision mesh filename=package://robotiq_85_description/meshes/collision/robotiq_8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; visual mesh filename=package://robotiq_85_description/meshes/visual/robotiq_85_i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
- added link robotiq_85_left_knuckle_link, mass 0.018491; collision mesh filename=package://robotiq_85_description/meshes/collision/robotiq_8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; visual mesh filename=package://robotiq_85_description/meshes/visual/robotiq_85_k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
- added link robotiq_85_right_finger_link, mass 0.027309; collision mesh filename=package://robotiq_85_description/meshes/collision/robotiq_8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; visual mesh filename=package://robotiq_85_description/meshes/visual/robotiq_85_f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
- added link robotiq_85_right_finger_tip_link, mass 0.019555; collision mesh filename=package://robotiq_85_description/meshes/collision/robotiq_8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; visual mesh filename=package://robotiq_85_description/meshes/visual/robotiq_85_f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
- added link robotiq_85_right_inner_knuckle_link, mass 0.029951; collision mesh filename=package://robotiq_85_description/meshes/collision/robotiq_8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; visual mesh filename=package://robotiq_85_description/meshes/visual/robotiq_85_i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
- added link robotiq_85_right_knuckle_link, mass 0.018491; collision mesh filename=package://robotiq_85_description/meshes/collision/robotiq_8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; visual mesh filename=package://robotiq_85_description/meshes/visual/robotiq_85_k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
- added link tool0
Joints:
- removed joint simple_arm_base_link-base
- removed joint simple_arm_joint_1
- removed joint simple_arm_joint_2
- removed joint simple_arm_joint_3
- removed joint simple_arm_joint_4
- removed joint simple_arm_joint_5
- removed joint simple_arm_joint_6
- removed joint simple_arm_joint_6-flange
- removed joint simple_arm_link_6-tool0
- removed joint simple_gripper_robotiq_85_base_joint
- removed joint simple_gripper_robotiq_85_left_finger_joint
- removed joint simple_gripper_robotiq_85_left_finger_tip_joint
- removed joint simple_gripper_robotiq_85_left_inner_knuckle_joint
- removed joint simple_gripper_robotiq_85_left_knuckle_joint
- removed joint simple_gripper_robotiq_85_right_finger_joint
- removed joint simple_gripper_robotiq_85_right_finger_tip_joint
- removed joint simple_gripper_robotiq_85_right_inner_knuckle_joint
- removed joint simple_gripper_robotiq_85_right_knuckle_joint
- removed joint world_joint
- added joint base_link-base: type fixed, parent base_link, child base, origin xyz=0 0 0 rpy=0 0 0
- added joint joint_1: type revolute, parent base_link, child link_1, origin xyz=0 0 0 rpy=0 0 0, axis 0 0 1, limit lower=-2.87979 upper=2.87979 effort=0 velocity=4.36332
- added joint joint_2: type revolute, parent link_1, child link_2, origin xyz=0 0 0.29 rpy=0 0 0, axis 0 1 0, limit lower=-1.91986 upper=1.91986 effort=0 velocity=4.36332
- added joint joint_3: type revolute, parent link_2, child link_3, origin xyz=0 0 0.27 rpy=0 0 0, axis 0 1 0, limit lower=-1.91986 upper=1.22173 effort=0 velocity=4.36332
- added joint joint_4: type revolute, parent link_3, child link_4, origin xyz=0 0 0.07 rpy=0 0 0, axis 1 0 0, limit lower=-2.79253 upper=2.79253 effort=0 velocity=5.58505
- added joint joint_5: type revolute, parent link_4, child link_5, origin xyz=0.302 0 0 rpy=0 0 0, axis 0 1 0, limit lower=-2.094395 upper=2.094395 effort=0 velocity=5.58505
- added joint joint_6: type revolute, parent link_5, child link_6, origin xyz=0.072 0 0 rpy=0 0 0, axis 1 0 0, limit lower=-6.98132 upper=6.98132 effort=0 velocity=7.33038
- added joint joint_6-flange: type fixed, parent link_6, child flange, origin xyz=0 0 0 rpy=0 0 0
- added joint link_6-tool0: type fixed, parent flange, child tool0, origin xyz=0 0 0 rpy=0 1.5707963267948966 0
- added joint robotiq_85_base_joint: type fixed, parent tool0, child robotiq_85_base_link, origin xyz=0 0 0 rpy=0 -1.570795 0
- added joint robotiq_85_left_finger_joint: type continuous, parent robotiq_85_left_knuckle_link, child robotiq_85_left_finger_link, origin xyz=-0.00408552455 -0.03148604435 0.0 rpy=0 0 0
- added joint robotiq_85_left_finger_tip_joint: type continuous, parent robotiq_85_left_inner_knuckle_link, child robotiq_85_left_finger_tip_link, origin xyz=0.04303959807 -0.03759940821 0.0 rpy=0.0 0.0 0.0, axis 0 0 1, limit lower=-3.14 upper=3.14 effort=0.1 velocity=100.0, mimic joint=robotiq_85_left_knuckle_joint multiplier=-1
- added joint robotiq_85_left_inner_knuckle_joint: type continuous, parent robotiq_85_base_link, child robotiq_85_left_inner_knuckle_link, origin xyz=0.06142 0.0127 0 rpy=3.14159 0.0 0.0, axis 0 0 1, limit lower=-3.14 upper=3.14 effort=0.1 velocity=100.0, mimic joint=robotiq_85_left_knuckle_joint offset=0
- added joint robotiq_85_left_knuckle_joint: type revolute, parent robotiq_85_base_link, child robotiq_85_left_knuckle_link, origin xyz=0.05490451627 0.03060114443 0.0 rpy=3.14159 0.0 0.0, axis 0 0 1, limit lower=0.0 upper=0.804 effort=1000 velocity=2.0
- added joint robotiq_85_right_finger_joint: type continuous, parent robotiq_85_right_knuckle_link, child robotiq_85_right_finger_link, origin xyz=-0.00408552455 -0.03148604435 0.0 rpy=0 0 0
- added joint robotiq_85_right_finger_tip_joint: type continuous, parent robotiq_85_right_inner_knuckle_link, child robotiq_85_right_finger_tip_link, origin xyz=0.04303959807 -0.03759940821  0.0 rpy=0.0 0.0 0.0, axis 0 0 1, limit lower=-3.14 upper=3.14 effort=0.1 velocity=100.0, mimic joint=robotiq_85_left_knuckle_joint multiplier=-1
- added joint robotiq_85_right_inner_knuckle_joint: type continuous, parent robotiq_85_base_link, child robotiq_85_right_inner_knuckle_link, origin xyz=0.06142 -0.0127 0 rpy=0 0 0, axis 0 0 1, limit lower=-3.14 upper=3.14 effort=0.1 velocity=100.0, mimic joint=robotiq_85_left_knuckle_joint offset=0
- added joint robotiq_85_right_knuckle_joint: type continuous, parent robotiq_85_base_link, child robotiq_85_right_knuckle_link, origin xyz=0.05490451627 -0.03060114443 0.0 rpy=0.0 0.0 0.0, axis 0 0 1, limit lower=-3.14 upper=3.14 effort=1000 velocity=100.0, mimic joint=robotiq_85_left_knuckle_joint
- added joint world-base_link-fixed: type fixed, parent world, child base_link
